File: pingpong_1d/electric_circuit.brd (EAGLE design)
At the start: 202.3 x 128.2 mm, 8 parts, among them U1 ARDUINO-UNO-R3-SHIELD, U2 LCD-16X2JHD-162A

Commit message: update circuit
Connections:
- net U1_D8: now also RRESISTANCE_BOUTON_GAUCHE.2, S1.3, S1.4; no longer RRESISTANCE_DROITE.2, S2.3, S2.4
- net U1_D9: now also RRESISTANCE_DROITE.2, S2.3, S2.4; no longer RRESISTANCE_BOUTON_GAUCHE.2, S1.3, S1.4
Changed lines of the file:
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@@
 </elements>
 <signals>
-<signal name="U1_D9">
+<signal name="U1_D8">
 <contactref element="S1" pad="3"/>
-<contactref element="U1" pad="D9"/>
 <contactref element="RRESISTANCE_BOUTON_GAUCHE" pad="2"/>
+<contactref element="U1" pad="D8"/>
 <contactref element="S1" pad="4"/>
 <wire x1="127.1142" y1="95.1765" x2="127.1142" y2="101.6789" width="0" layer="19" extent="1-1"/>
 <wire x1="127.1142" y1="95.1765" x2="127.3936" y2="86.9977" width="0" layer="19" extent="1-1"/>
-<wire x1="66.8399" y1="122.4937" x2="127.1142" y2="101.6789" width="0" layer="19" extent="1-1"/>
+<wire x1="69.3799" y1="122.4937" x2="127.1142" y2="101.6789" width="0" layer="19" extent="1-1"/>
 </signal>
 <signal name="U1_GND">
@@
 <wire x1="37.084" y1="36.6268" x2="78.2699" y2="122.4937" width="0" layer="19" extent="1-1"/>
 </signal>
-<signal name="U1_D8">
+<signal name="U1_D9">
 <contactref element="S2" pad="4"/>
 <contactref element="RRESISTANCE_DROITE" pad="2"/>
 <contactref element="S2" pad="3"/>
-<contactref element="U1" pad="D8"/>
+<contactref element="U1" pad="D9"/>
 <wire x1="195.6942" y1="101.6789" x2="195.6942" y2="95.1765" width="0" layer="19" extent="1-1"/>
 <wire x1="195.9736" y1="86.9977" x2="195.6942" y2="95.1765" width="0" layer="19" extent="1-1"/>
-<wire x1="195.6942" y1="101.6789" x2="69.3799" y2="122.4937" width="0" layer="19" extent="1-1"/>
+<wire x1="195.6942" y1="101.6789" x2="66.8399" y2="122.4937" width="0" layer="19" extent="1-1"/>
 </signal>
 </signals>
